File: LetsTry Button.kicad_pcb (KiCad board)
At the start: 2 copper layers, 81.8 x 85.9 mm, 36 parts, among them J1 Screw_Terminal_01x02, J2 Screw_Terminal_01x02, J22 Screw_Terminal_01x08, J3 Screw_Terminal_01x03, J7 Screw_Terminal_01x08, J9 Screw_Terminal_01x02, P2 RB1-125BAG1A, P3 USB_C_Plug, U1 W5100, U2 ESP32-S3-DEVKITC-1-N8R2

Commit message: Add files via upload
Connections:
- net Net-(J22-Pin_1) renamed /W5100/5V
- J7 pad 3: /W5100/CS -> Net-(J7-Pin_3)
- U1 pad 55: /W5100/GPIO15 -> /W5100/CS
- U2 pad J1_10: Net-(J7-Pin_6) -> Net-(J22-Pin_6)
- U2 pad J1_11: Net-(J7-Pin_7) -> Net-(J22-Pin_7)
- U2 pad J1_12: unconnected-(U2-GPIO8-PadJ1_12) -> Net-(J22-Pin_8)
- U2 pad J1_15: Net-(J3-Pin_2) -> unconnected-(U2-GPIO9-PadJ1_15)
- U2 pad J1_16: /W5100/CS -> unconnected-(U2-GPIO10-PadJ1_16)
- U2 pad J1_17: Net-(J7-Pin_4) -> unconnected-(U2-GPIO11-PadJ1_17)
- U2 pad J1_6: Net-(J1-Pin_2) -> Net-(J22-Pin_3)
- U2 pad J1_7: Net-(J9-Pin_2) -> Net-(J22-Pin_4)
- U2 pad J1_8: /W5100/GPIO15 -> /W5100/CS
- U2 pad J1_9: Net-(J7-Pin_5) -> Net-(J22-Pin_5)
- U2 pad J3_10: Net-(J22-Pin_5) -> Net-(J9-Pin_2)
- U2 pad J3_11: Net-(J22-Pin_4) -> Net-(J3-Pin_2)
- U2 pad J3_12: Net-(J22-Pin_3) -> Net-(J1-Pin_2)
- U2 pad J3_15: Net-(J22-Pin_6) -> unconnected-(U2-GPIO45-PadJ3_15)
- U2 pad J3_16: Net-(J22-Pin_8) -> unconnected-(U2-GPIO48-PadJ3_16)
- U2 pad J3_17: Net-(J22-Pin_7) -> unconnected-(U2-GPIO47-PadJ3_17)
- U2 pad J3_18: Net-(J7-Pin_8) -> unconnected-(U2-GPIO21-PadJ3_18)
- U2 pad J3_2: unconnected-(U2-U0TXD/GPIO43-PadJ3_2) -> Net-(J7-Pin_3)
- U2 pad J3_3: unconnected-(U2-U0RXD/GPIO44-PadJ3_3) -> Net-(J7-Pin_4)
- U2 pad J3_6: unconnected-(U2-MTMS/GPIO42-PadJ3_6) -> Net-(J7-Pin_5)
- U2 pad J3_7: unconnected-(U2-MTDI/GPIO41-PadJ3_7) -> Net-(J7-Pin_6)
- U2 pad J3_8: unconnected-(U2-MTDO/GPIO40-PadJ3_8) -> Net-(J7-Pin_7)
- U2 pad J3_9: unconnected-(U2-MTCK/GPIO39-PadJ3_9) -> Net-(J7-Pin_8)
Routing:
- net /W5100/CS: track 93.9 -> 25.4 mm
- net Net-(J7-Pin_4): track 59.7 -> 23.3 mm, vias 2 -> 0
- net Net-(J22-Pin_3): track 87.7 -> 56.7 mm, vias 1 -> 0
- net Net-(J22-Pin_7): track 92.9 -> 62.1 mm, vias 1 -> 0
- net Net-(J1-Pin_2): track 38.9 -> 69.6 mm
- net Net-(J22-Pin_6): track 89.6 -> 61.5 mm
- net Net-(J22-Pin_4): track 86.5 -> 58.4 mm, vias 1 -> 0
- net Net-(J22-Pin_8): track 90.9 -> 63.8 mm
- net /W5100/GPIO15: track 25.5 -> 0.00 mm, vias 1 -> 0
- net Net-(J22-Pin_5): track 84.5 -> 60.6 mm
- net Net-(J7-Pin_8): track 65.6 -> 42.8 mm
- net Net-(J7-Pin_3): track 0.00 -> 19.7 mm
- net Net-(J9-Pin_2): track 31.9 -> 49.4 mm
- net /W5100/5V: track 181.6 -> 166.6 mm
- net Net-(J7-Pin_7): track 49.0 -> 39.2 mm, vias 1 -> 0
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
Commit message: Add files via upload
usbc
Parts:
- removed J22, J7: Screw_Terminal_01x08, termsag:TE_282834-8
- added J4: 1658525-8, moreterms:TE_1658525-8, F.Cu at (147.6, 153.2)
- moved R3 83.0 mm to (151.8, 60.8), turned to 90 degrees
- moved P3 73.2 mm to (147.3, 101.6), turned to 90 degrees
- moved P2 64.8 mm to (147.3, 72.0), turned to 90 degrees
- moved R1 64.1 mm to (149.1, 83.3), turned to -90 degrees
- moved C3 62.1 mm to (136.5, 59.3), turned to -90 degrees
- moved R13 59.1 mm to (137.2, 61.8), turned to -90 degrees
- moved R12 57.4 mm to (135.9, 61.8), turned to -90 degrees
- moved J2 57.4 mm to (148.8, 90.4), turned to -90 degrees
- moved H4 52.9 mm to (168.7, 191.5)
- moved J1 49.3 mm to (147.3, 133.6), turned to 90 degrees
- moved R2 47.0 mm to (140.5, 81.4), turned to 90 degrees
- moved C2 45.9 mm to (140.0, 84.5), turned to 90 degrees
- moved R11 45.1 mm to (141.7, 121.9), turned to 0 degrees
- moved R4 45.0 mm to (139.4, 81.4), turned to 90 degrees
- moved C1 36.4 mm to (135.3, 83.4), turned to -90 degrees
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Connections:
- net /W5100/5V renamed Net-(J3-Pin_1)
- P3 pad A6: unconnected-(P3-D+-PadA6) -> Net-(P3-D+)
- P3 pad A7: unconnected-(P3-D--PadA7) -> Net-(P3-D-)
- U2 pad J1_14: unconnected-(U2-GPIO46-PadJ1_14) -> Net-(J3-Pin_2)
- U2 pad J1_15: unconnected-(U2-GPIO9-PadJ1_15) -> Net-(J9-Pin_2)
- U2 pad J3_10: Net-(J9-Pin_2) -> Net-(J1-Pin_2)
- U2 pad J3_11: Net-(J3-Pin_2) -> unconnected-(U2-GPIO37-PadJ3_11)
- U2 pad J3_12: Net-(J1-Pin_2) -> unconnected-(U2-GPIO36-PadJ3_12)
- U2 pad J3_16: unconnected-(U2-GPIO48-PadJ3_16) -> GND
- U2 pad J3_19: unconnected-(U2-USB_D+/GPIO20-PadJ3_19) -> Net-(P3-D+)
- U2 pad J3_20: unconnected-(U2-USB_D-/GPIO19-PadJ3_20) -> Net-(P3-D-)
Routing:
- net Net-(J3-Pin_1): track 166.6 -> 36.3 mm
- net /W5100/GPIO12: track 22.5 -> 89.7 mm
- net /W5100/GPIO13: track 26.8 -> 84.3 mm
- net /W5100/CS: track 25.4 -> 82.3 mm, vias 0 -> 2
- net Net-(J3-Pin_2): track 59.4 -> 12.8 mm
- net Net-(J9-Pin_2): track 49.4 -> 10.7 mm
- net /W5100/GPIO14: track 31.3 -> 66.9 mm
- net Net-(J1-Pin_2): track 69.6 -> 34.6 mm
- net Net-(U2-GPIO8): track 63.8 -> 34.0 mm
- net Net-(P3-D+): track 0.00 -> 28.7 mm
- net Net-(P3-D-): track 0.00 -> 28.1 mm
- net Net-(U2-GPIO18): track 62.1 -> 34.0 mm
- net Net-(U2-GPIO17): track 61.5 -> 34.0 mm
- net Net-(U2-GPIO7): track 58.4 -> 31.5 mm
- net Net-(U2-GPIO16): track 60.6 -> 34.0 mm
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Other:
- board size 81.8 x 85.9 mm -> 128.6 x 144.6 mm

Commit message: Add files via upload
Parts:
- added D3: SP0503BAHT, Package_TO_SOT_SMD:SOT-143, F.Cu at (141.8, 102.1)
- P3: footprint Connector_USB:USB_C_Receptacle_Amphenol_12401548E4-2A -> Connector_USB:USB_C_Receptacle_Palconn_UTC16-G
- moved H3 41.5 mm to (109.2, 168.1)
- moved H1 38.9 mm to (107.7, 57.4)
- moved H4 30.2 mm to (148.3, 169.2)
- moved H2 17.6 mm to (150.4, 53.8)
- moved P3 0.59 mm to (147.6, 102.1)
Connections:
- net Net-(J2-Pin_2) renamed /W5100/VBUS
- net Net-(J3-Pin_2) renamed /W5100/GPIO46
- net Net-(J9-Pin_2) renamed /W5100/GPIO9
- net Net-(P3-D+) renamed /W5100/USB D+
- net Net-(P3-D-) renamed /W5100/USB D-
- net Net-(U2-GPIO16) renamed /W5100/GPIO16
- net Net-(U2-GPIO17) renamed /W5100/GPIO17
- net Net-(U2-GPIO18) renamed /W5100/GPIO18
- net Net-(U2-GPIO6) renamed /W5100/GPIO6
- net Net-(U2-GPIO7) renamed /W5100/GPIO7
- net Net-(U2-GPIO8) renamed /W5100/GPIO8
- net Net-(U2-MTCK/GPIO39) renamed /W5100/GPIO39
- net Net-(U2-MTDI/GPIO41) renamed /W5100/GPIO41
- net Net-(U2-MTDO/GPIO40) renamed /W5100/GPIO40
- net Net-(U2-MTMS/GPIO42) renamed /W5100/GPIO42
- net Net-(U2-U0RXD/GPIO44) renamed /W5100/GPIO44
- net Net-(U2-U0TXD/GPIO43) renamed /W5100/GPIO43
- C1 pad 1: 3.3V -> +3.3V
- J2 pad 1: 3.3V -> +3.3V
- J3 pad 1: Net-(J3-Pin_1) -> /W5100/5V
- J4 pad 16: 3.3V -> /W5100/5V
- J4 pad 8: 3.3V -> +3.3V
- J9 pad 1: Net-(J3-Pin_1) -> /W5100/5V
- P2 pad R3: 3.3V -> +3.3V
- P2 pad R6: 3.3V -> +3.3V
- R1 pad 2: 3.3V -> +3.3V
- R10 pad 2: 3.3V -> +3.3V
- R11 pad 1: Net-(J3-Pin_1) -> /W5100/5V
- R3 pad 2: 3.3V -> +3.3V
- R5 pad 2: 3.3V -> +3.3V
- R6 pad 2: 3.3V -> +3.3V
- R7 pad 2: 3.3V -> +3.3V
- R8 pad 2: 3.3V -> +3.3V
- R9 pad 2: 3.3V -> +3.3V
- U1 pad 12: 3.3V -> +3.3V
- U1 pad 18: 3.3V -> +3.3V
- U1 pad 2: 3.3V -> +3.3V
- U1 pad 44: 3.3V -> +3.3V
- U2 pad J1_1: 3.3V -> +3.3V
- U2 pad J1_2: 3.3V -> +3.3V
- U2 pad J1_21: Net-(J3-Pin_1) -> /W5100/5V
- U2 pad J3_16: GND -> unconnected-(U2-GPIO48-PadJ3_16)
Routing:
- net 3.3V: track 234.1 -> 0.00 mm, vias 4 -> 0
- net +3.3V: track 0.00 -> 228.6 mm, vias 0 -> 4
- net /W5100/5V: track 0.00 -> 61.7 mm
- net Net-(J3-Pin_1): track 36.3 -> 0.00 mm
- net GND: track 51.0 -> 31.6 mm, vias 8 -> 13
- net /W5100/VBUS: track 22.8 -> 27.8 mm
- net /W5100/CS: track 82.3 -> 78.1 mm
- net /W5100/USB D-: track 28.1 -> 31.4 mm
- net /W5100/USB D+: track 28.7 -> 31.5 mm
- net /W5100/GPIO12: track 89.7 -> 87.6 mm
- net /W5100/GPIO14: track 66.9 -> 64.8 mm
- net /W5100/GPIO13: track 84.3 -> 82.5 mm
- net (no net): track 0.64 -> 0.00 mm
Other:
- board size 128.6 x 144.6 mm -> 51.8 x 124.5 mm

Commit message: Add files via upload
even new
Parts:
- moved H1 6.16 mm to (112.0, 53.0)
- moved H3 2.91 mm to (112.0, 169.0)
- moved J3 2.54 mm to (149.9, 123.4)
- moved J4 2.03 mm to (149.6, 153.2)
- moved H2 1.61 mm to (149.0, 53.0)
- moved J1 1.52 mm to (148.8, 133.6)
- moved J9 1.52 mm to (148.8, 113.3)
- moved H4 0.68 mm to (149.0, 169.0)
Routing:
- net /W5100/GPIO46: track 12.8 -> 15.3 mm
- net /W5100/GPIO8: track 34.0 -> 36.5 mm
- net /W5100/GPIO17: track 34.0 -> 36.2 mm
- net /W5100/GPIO42: track 42.2 -> 44.2 mm
- net /W5100/GPIO16: track 34.0 -> 36.1 mm
- net /W5100/GPIO7: track 31.5 -> 33.5 mm
- net /W5100/GPIO6: track 40.3 -> 42.4 mm
- net /W5100/GPIO44: track 38.0 -> 40.1 mm
- net /W5100/GPIO43: track 38.0 -> 40.1 mm
- net /W5100/GPIO41: track 42.8 -> 44.8 mm
- net /W5100/GPIO40: track 41.9 -> 43.9 mm
- net /W5100/GPIO39: track 41.3 -> 43.3 mm
- net /W5100/GPIO18: track 34.0 -> 36.1 mm
- net Net-(J1-Pin_2): track 34.6 -> 36.1 mm
- net /W5100/GPIO9: track 10.7 -> 12.2 mm
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Other:
- board size 51.8 x 124.5 mm -> 47.2 x 126.5 mm
