File: LetsTry Button.kicad_pcb (KiCad board)
At the start: 2 copper layers, 128.6 x 144.6 mm, 35 parts, among them J1 Screw_Terminal_01x02, J2 Screw_Terminal_01x02, J3 Screw_Terminal_01x03, J4 1658525-8, J9 Screw_Terminal_01x02, P2 RB1-125BAG1A, P3 USB_C_Plug, U1 W5100, U2 ESP32-S3-DEVKITC-1-N8R2

Commit message: Add files via upload
fixed
Parts:
- removed R11: 100k, Resistor_SMD:R_0402_1005Metric
- added D3: SP0503BAHT, Package_TO_SOT_SMD:SOT-143, F.Cu at (141.8, 102.1)
- P3: footprint Connector_USB:USB_C_Receptacle_Amphenol_12401548E4-2A -> Connector_USB:USB_C_Receptacle_Palconn_UTC16-G
- moved H3 44.2 mm to (112.0, 169.0)
- moved H1 43.9 mm to (112.0, 53.0)
- moved H4 29.9 mm to (149.0, 169.0)
- moved J4 21.6 mm to (130.2, 166.0), turned to 0 degrees
- moved H2 19.2 mm to (149.0, 53.0)
- moved J3 2.54 mm to (149.9, 123.4)
- moved J1 1.52 mm to (148.8, 133.6)
- moved J9 1.52 mm to (148.8, 113.3)
- moved P3 0.59 mm to (147.6, 102.1)
Connections:
- net Net-(J2-Pin_2) renamed /W5100/VBUS
- net Net-(J3-Pin_2) renamed /W5100/GPIO46
- net Net-(J9-Pin_2) renamed /W5100/GPIO9
- net Net-(P3-D+) renamed /W5100/USB D+
- net Net-(P3-D-) renamed /W5100/USB D-
- net Net-(U2-MTCK/GPIO39) renamed /W5100/GPIO39
- net Net-(U2-MTDI/GPIO41) renamed /W5100/GPIO41
- net Net-(U2-MTDO/GPIO40) renamed /W5100/GPIO40
- net Net-(U2-MTMS/GPIO42) renamed /W5100/GPIO42
- net Net-(U2-U0RXD/GPIO44) renamed /W5100/GPIO44
- net Net-(U2-U0TXD/GPIO43) renamed /W5100/GPIO43
- C1 pad 1: 3.3V -> +3.3V
- J1 pad 1: Net-(J1-Pin_1) -> +3.3V
- J2 pad 1: 3.3V -> +5V
- J3 pad 1: Net-(J3-Pin_1) -> +5V
- J4 pad 10: Net-(U2-GPIO7) -> /W5100/GPIO18
- J4 pad 11: Net-(U2-GPIO16) -> /W5100/GPIO17
- J4 pad 12: Net-(U2-GPIO17) -> /W5100/GPIO16
- J4 pad 13: Net-(U2-GPIO18) -> /W5100/GPIO7
- J4 pad 14: Net-(U2-GPIO8) -> /W5100/GPIO6
- J4 pad 16: 3.3V -> +5V
- J4 pad 8: 3.3V -> +3.3V
- J4 pad 9: Net-(U2-GPIO6) -> /W5100/GPIO8
- J9 pad 1: Net-(J3-Pin_1) -> +3.3V
- P2 pad R3: 3.3V -> +3.3V
- P2 pad R6: 3.3V -> +3.3V
- R1 pad 2: 3.3V -> +3.3V
- R10 pad 2: 3.3V -> +3.3V
- R3 pad 2: 3.3V -> +3.3V
- R5 pad 2: 3.3V -> +3.3V
- R6 pad 2: 3.3V -> +3.3V
- R7 pad 2: 3.3V -> +3.3V
- R8 pad 2: 3.3V -> +3.3V
- R9 pad 2: 3.3V -> +3.3V
- U1 pad 12: 3.3V -> +3.3V
- U1 pad 18: 3.3V -> +3.3V
- U1 pad 2: 3.3V -> +3.3V
- U1 pad 44: 3.3V -> +3.3V
- U2 pad J1_1: 3.3V -> +3.3V
- U2 pad J1_10: Net-(U2-GPIO17) -> /W5100/GPIO17
- U2 pad J1_11: Net-(U2-GPIO18) -> /W5100/GPIO18
- U2 pad J1_12: Net-(U2-GPIO8) -> /W5100/GPIO8
- U2 pad J1_2: 3.3V -> +3.3V
- U2 pad J1_21: Net-(J3-Pin_1) -> +5V
- U2 pad J1_6: Net-(U2-GPIO6) -> /W5100/GPIO6
- U2 pad J1_7: Net-(U2-GPIO7) -> /W5100/GPIO7
- U2 pad J1_9: Net-(U2-GPIO16) -> /W5100/GPIO16
- U2 pad J3_16: GND -> unconnected-(U2-GPIO48-PadJ3_16)
Routing:
- net +3.3V: track 0.00 -> 257.5 mm, vias 0 -> 2
- net 3.3V: track 234.1 -> 0.00 mm, vias 4 -> 0
- net +5V: track 0.00 -> 116.2 mm
- net /W5100/GPIO8: track 0.00 -> 53.1 mm
- net /W5100/GPIO18: track 0.00 -> 49.9 mm
- net /W5100/GPIO17: track 0.00 -> 45.9 mm
- net /W5100/GPIO16: track 0.00 -> 42.3 mm
- net Net-(U2-GPIO6): track 40.3 -> 0.00 mm
- net Net-(J3-Pin_1): track 36.3 -> 0.00 mm
- net /W5100/GPIO7: track 0.00 -> 36.2 mm
- net Net-(U2-GPIO16): track 34.0 -> 0.00 mm
- net Net-(U2-GPIO8): track 34.0 -> 0.00 mm
- net Net-(U2-GPIO18): track 34.0 -> 0.00 mm
- net Net-(U2-GPIO17): track 34.0 -> 0.00 mm
- net /W5100/GPIO6: track 0.00 -> 32.6 mm
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Other:
- board size 128.6 x 144.6 mm -> 47 x 126 mm
- board text added: "3.3V"
- board text added: "5V"
- board text added: "GND"
- board text added: "GPIO16"
- board text added: "GPIO17"
- board text added: "GPIO18"
- board text added: "GPIO39"
- board text added: "GPIO40"
- board text added: "GPIO41"
- board text added: "GPIO42"
- board text added: "GPIO44"
- board text added: "GPIO45"
- board text added: "GPIO6"
- board text added: "GPIO7"
- board text added: "GPIO8"

Commit message: Add files via upload
Parts:
- R1, R3: value 330 -> 470
- moved H3 4.00 mm to (112.0, 173.0)
- moved H4 4.00 mm to (149.0, 173.0)
- moved J4 1.50 mm to (130.1, 167.5)
Routing:
- net +5V: track 116.2 -> 119.3 mm
- net /W5100/GPIO6: track 32.6 -> 34.2 mm
- net /W5100/GPIO7: track 36.2 -> 37.8 mm
- net /W5100/GPIO8: track 53.1 -> 54.7 mm
- net /W5100/GPIO18: track 49.9 -> 51.5 mm
- net /W5100/GPIO17: track 45.9 -> 47.5 mm
- net /W5100/GPIO16: track 42.3 -> 43.9 mm
- net /W5100/GPIO41: track 37.0 -> 38.4 mm
- net /W5100/GPIO44: track 24.7 -> 26.2 mm
- net /W5100/GPIO42: track 33.4 -> 34.8 mm
- net /W5100/GPIO40: track 40.5 -> 42.0 mm
- net +3.3V: track 257.5 -> 258.9 mm
- net /W5100/GPIO43: track 21.1 -> 22.6 mm
- net /W5100/GPIO39: track 44.1 -> 45.6 mm
Other:
- board size 47 x 126 mm -> 47 x 130 mm
