File: LetsTry Button.kicad_pcb (KiCad board)
At the start: 2 copper layers, 47 x 130 mm, 35 parts, among them J1 Screw_Terminal_01x02, J2 Screw_Terminal_01x02, J3 Screw_Terminal_01x03, J4 1658525-8, J9 Screw_Terminal_01x02, P2 RB1-125BAG1A, P3 USB_C_Plug, U1 W5100, U2 ESP32-S3-DEVKITC-1-N8R2

Commit message: i finally learnt how to use github. Final Buttton?
Parts:
- moved J4 25.4 mm to (150.5, 152.4), turned to 90 degrees
- moved H3 5.00 mm to (112.0, 168.0)
- moved H4 5.00 mm to (149.0, 168.0)
- moved J1 1.16 mm to (150.0, 133.6)
Connections:
- J4 pad 10: /W5100/GPIO18 -> /W5100/GPIO7
- J4 pad 11: /W5100/GPIO17 -> /W5100/GPIO16
- J4 pad 12: /W5100/GPIO16 -> /W5100/GPIO17
- J4 pad 13: /W5100/GPIO7 -> /W5100/GPIO18
- J4 pad 14: /W5100/GPIO6 -> /W5100/GPIO8
- J4 pad 9: /W5100/GPIO8 -> /W5100/GPIO6
Routing:
- net +5V: track 119.3 -> 85.9 mm
- net /W5100/GPIO8: track 54.7 -> 34.4 mm
- net +3.3V: track 258.9 -> 240.1 mm
- net /W5100/GPIO43: track 22.6 -> 40.6 mm
- net /W5100/GPIO18: track 51.5 -> 35.1 mm
- net /W5100/GPIO44: track 26.2 -> 40.6 mm
- net /W5100/GPIO17: track 47.5 -> 34.6 mm
- net /W5100/GPIO16: track 43.9 -> 34.7 mm
- net /W5100/GPIO42: track 34.8 -> 42.7 mm
- net /W5100/GPIO7: track 37.8 -> 32.0 mm
- net /W5100/GPIO41: track 38.4 -> 42.7 mm
- net /W5100/GPIO39: track 45.6 -> 42.9 mm
- net /W5100/GPIO6: track 34.2 -> 31.9 mm
- net Net-(J1-Pin_2): track 37.1 -> 38.2 mm
- net /W5100/GPIO40: track 42.0 -> 42.7 mm
Other:
- board size 47 x 130 mm -> 47 x 125 mm
- board text added: "16"
- board text added: "17"
- board text added: "18"
- board text added: "39"
- board text added: "40"
- board text added: "41"
- board text added: "42"
- board text added: "44"
- board text added: "45"
- board text added: "6"
- board text added: "7"
- board text added: "8"
- board text removed: "GPIO16"
- board text removed: "GPIO17"
- board text removed: "GPIO18"
- board text removed: "GPIO39"
- board text removed: "GPIO40"
- board text removed: "GPIO41"
- board text removed: "GPIO42"
- board text removed: "GPIO44"
- board text removed: "GPIO45"
- board text removed: "GPIO6"
- board text removed: "GPIO7"
- board text removed: "GPIO8"

Commit message: update
Parts:
- removed P3: USB_C_Plug, Connector_USB:USB_C_Receptacle_Palconn_UTC16-G
- added J5: USB_C_Receptacle_USB2.0, Connector_USB:USB_C_Receptacle_Palconn_UTC16-G, F.Cu at (148.4, 102.1)
- added R11: 10k, Resistor_SMD:R_0402_1005Metric, F.Cu at (122.6, 62.3)
- added R14: 12.3k, Resistor_SMD:R_0603_1608Metric, F.Cu at (132.9, 76.2)
- added R15: 5.1k, Resistor_SMD:R_0402_1005Metric, F.Cu at (143.9, 103.8)
- added R16: 5.1k, Resistor_SMD:R_0402_1005Metric, F.Cu at (143.9, 99.6)
- added TP1: TestPoint, TestPoint:TestPoint_Pad_D1.0mm, F.Cu at (116.8, 70.2)
- added TP2: TestPoint, TestPoint:TestPoint_Pad_D1.0mm, F.Cu at (116.8, 72.2)
- added TP3: TestPoint, TestPoint:TestPoint_Pad_D1.0mm, F.Cu at (116.8, 74.2)
- moved D3 0.52 mm to (142.1, 101.7), turned to -90 degrees
Connections:
- net /W5100/GPIO14 renamed /W5100/SCLK
- U1 pad 1: unconnected-(U1-RSET_BG-Pad1) -> Net-(U1-RSET_BG)
- U1 pad 27: /W5100/GPIO12 -> /W5100/MISO
- U1 pad 28: /W5100/GPIO13 -> /W5100/MOSI
- U1 pad 29: unconnected-(U1-~{SCS}-Pad29) -> /W5100/CS
- U1 pad 31: unconnected-(U1-SEN-Pad31) -> Net-(U1-SEN)
- U1 pad 55: /W5100/CS -> Net-(U1-~{CS})
- U1 pad 57: unconnected-(U1-~{WR}-Pad57) -> Net-(U1-~{WR})
- U1 pad 58: unconnected-(U1-~{RD}-Pad58) -> Net-(U1-~{RD})
- U2 pad J1_17: unconnected-(U2-GPIO11-PadJ1_17) -> /W5100/MISO
- U2 pad J1_18: /W5100/GPIO12 -> /W5100/MOSI
- U2 pad J1_19: /W5100/GPIO13 -> /W5100/CS
- U2 pad J1_8: /W5100/CS -> unconnected-(U2-GPIO15-PadJ1_8)
Routing:
- net /W5100/GPIO12: track 87.6 -> 0.00 mm
- net /W5100/MISO: track 0.00 -> 86.3 mm
- net /W5100/GPIO13: track 82.5 -> 0.00 mm
- net /W5100/MOSI: track 0.00 -> 82.4 mm
- net /W5100/USB D+: track 31.5 -> 40.4 mm
- net /W5100/VBUS: track 27.8 -> 19.4 mm
- net +3.3V: track 240.1 -> 247.2 mm
- net /W5100/USB D-: track 31.4 -> 35.6 mm
- net Net-(U1-RSET_BG): track 0.00 -> 3.70 mm
- net Net-(U1-~{RD}): track 0.00 -> 3.19 mm
- net Net-(U1-~{CS}): track 0.00 -> 2.47 mm
- net Net-(U1-SEN): track 0.00 -> 2.18 mm
- net Net-(U1-~{WR}): track 0.00 -> 2.07 mm
- net /W5100/CS: track 76.5 -> 78.4 mm, vias 1 -> 0
- net Net-(J5-CC2): track 0.00 -> 1.83 mm
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