File: W5100s.kicad_sch (KiCad schematic)
At the start: 31 parts, among them J1 Screw_Terminal_01x02, J2 Screw_Terminal_01x02, J3 Screw_Terminal_01x03, J4 1658525-8, J9 Screw_Terminal_01x02, P1 RB1-125BAG1A, P1 USB_C_Plug, U3 W5100, U4 ESP32-S3-DEVKITC-1-N8R2

Commit message: Add files via upload
New one, idk if TVS diode is right
Parts:
- added D3: SP0503BAHT, Package_TO_SOT_SMD:SOT-143, symbol Power_Protection:SP0503BAHT
- P1: footprint Connector_USB:USB_C_Receptacle_Amphenol_12401548E4-2A -> Connector_USB:USB_C_Receptacle_Palconn_UTC16-G
Connections:
- net GND: now also D3.1 (A); no longer U4.J3_16 (GPIO48)
- net 5V: now reaches J3.1 (Pin_1), J9.1 (Pin_1), R25.1, U4.J1_21 (5V0)
- net 5V: now also J4.16
- net at U4.J1_14 (GPIO46): no longer J3.2 (Pin_2)
- net GPIO43: now reaches J4.1, U4.J3_2 (U0TXD/GPIO43)
- net GPIO7: now reaches J4.10, U4.J1_7 (GPIO7)
- net GPIO16: now reaches J4.11, U4.J1_9 (GPIO16)
- net GPIO17: now reaches J4.12, U4.J1_10 (GPIO17)
- net GPIO18: now reaches J4.13, U4.J1_11 (GPIO18)
- net GPIO8: now reaches J4.14, U4.J1_12 (GPIO8)
- net GPIO44: now reaches J4.2, U4.J3_3 (U0RXD/GPIO44)
- net GPIO42: now reaches J4.3, U4.J3_6 (MTMS/GPIO42)
- net GPIO41: now reaches J4.4, U4.J3_7 (MTDI/GPIO41)
- net GPIO40: now reaches J4.5, U4.J3_8 (MTDO/GPIO40)
- net GPIO39: now reaches J4.6, U4.J3_9 (MTCK/GPIO39)
- net GPIO6: now reaches J4.9, U4.J1_6 (GPIO6)
- net GPIO9: now reaches J9.2 (Pin_2), U4.J1_15 (GPIO9)
- net GPIO46: now reaches U4.J3_15 (GPIO45)
- net GPIO46: now also J3.2 (Pin_2)
- net USB D+: now reaches P1.A6 (D+), U4.J3_19 (USB_D+/GPIO20)
- net USB D+: now also D3.2 (K)
- net USB D-: now reaches P1.A7 (D-), U4.J3_20 (USB_D-/GPIO19)
- net USB D-: now also D3.3 (K)
- net VBUS: now reaches J2.2 (Pin_2), P1.A4 (VBUS), P1.A9 (VBUS), P1.B4 (VBUS), P1.B9 (VBUS)
- net VBUS: now also D3.4 (K)
- net 3.3V renamed +3.3V
- net +3.3V: no longer J4.16
Other:
- moved on the sheet: J2, J3, J4, J9

Commit message: Add files via upload
even new
Connections:
- net GPIO46: now also U4.J1_14 (GPIO46); no longer U4.J3_15 (GPIO45)
Changed lines of the file:
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@@
+    (stroke (width 0) (type default))
+  )
+  (wire (pts (xy 232.41 102.87) (xy 229.87 102.87))
     (stroke (width 0) (type default))
   )
@@
     (effects (font (size 1.27 1.27)) (justify left bottom))
   )
-  (label "GPIO46" (at 229.87 100.33 0) (fields_autoplaced)
-    (effects (font (size 1.27 1.27)) (justify left bottom))
-  )
+  (label "GPIO46" (at 232.41 102.87 0) (fields_autoplaced)
+    (effects (font (size 1.27 1.27)) (justify left bottom))
+  )
