File: W5100s.kicad_sch (KiCad schematic)
At the start: 32 parts, among them J1 Screw_Terminal_01x02, J2 Screw_Terminal_01x02, J3 Screw_Terminal_01x03, J4 1658525-8, J9 Screw_Terminal_01x02, P1 RB1-125BAG1A, P1 USB_C_Plug, U3 W5100, U4 ESP32-S3-DEVKITC-1-N8R2

Commit message: i fimally learnt how to use github
Parts:
- removed R25: 100k, Resistor_SMD:R_0402_1005Metric, symbol Device:R
- R17, R18: value 330 -> 470
Connections:
- net +3.3V: now also J1.1 (Pin_1), J9.1 (Pin_1); no longer J2.1 (Pin_1)
- net GPIO16: now also J4.12; no longer J4.11
- net GPIO17: now also J4.11; no longer J4.12
- net GPIO18: now also J4.10; no longer J4.13
- net GPIO46: now also U4.J1_14 (GPIO46); no longer U4.J3_15 (GPIO45)
- net GPIO6: now also J4.14; no longer J4.9
- net GPIO7: now also J4.13; no longer J4.10
- net GPIO8: now also J4.9; no longer J4.14
- net 5V renamed +5V
- net +5V: now also J2.1 (Pin_1); no longer J9.1 (Pin_1)
- no-connect marks 2 -> 3
