File: W5100s.kicad_sch (KiCad schematic)
At the start: 31 parts, among them J1 Screw_Terminal_01x02, J2 Screw_Terminal_01x02, J3 Screw_Terminal_01x03, J4 1658525-8, J9 Screw_Terminal_01x02, P1 RB1-125BAG1A, P1 USB_C_Plug, U3 W5100, U4 ESP32-S3-DEVKITC-1-N8R2

Commit message: update
Parts:
- removed P1: USB_C_Plug, Connector_USB:USB_C_Receptacle_Palconn_UTC16-G, symbol Connector:USB_C_Plug
- added J5: USB_C_Receptacle_USB2.0, Connector_USB:USB_C_Receptacle_Palconn_UTC16-G, symbol Connector:USB_C_Receptacle_USB2.0
- added R11: 10k, Resistor_SMD:R_0402_1005Metric, symbol Device:R_Small
- added R14: 12.3k, Resistor_SMD:R_0603_1608Metric, symbol Device:R_Small
- added R15, R16: 5.1k, Resistor_SMD:R_0402_1005Metric, symbol Device:R_Small
- added TP1, TP2, TP3: TestPoint, TestPoint:TestPoint_Pad_D1.0mm, symbol Connector:TestPoint
Connections:
- net +3.3V: now also R11.1
- net CS: now also U3.29 (~{SCS}), U4.J1_19 (GPIO13); no longer U3.55 (~{CS}), U4.J1_8 (GPIO15)
- net GND: now also J5.A1 (GND), J5.A12 (GND), J5.B1 (GND), J5.B12 (GND), J5.S1 (SHIELD), R14.2, R15.2, R16.2
- net USB D+: now also J5.A6 (D+), J5.B6 (D+)
- net USB D-: now also J5.A7 (D-), J5.B7 (D-)
- net VBUS: now also J5.A4 (VBUS), J5.A9 (VBUS), J5.B4 (VBUS), J5.B9 (VBUS)
- net at U3.1 (RSET_BG): now also R14.1
- net at U3.31 (SEN): now also R11.2
- net at U3.57 (~{WR}): now also TP2.1
- net at U3.58 (~{RD}): now also TP3.1
- net MISO: now reaches U4.J1_17 (GPIO11)
- net MISO: now also U3.27 (MISO)
- net GPIO12 renamed MOSI
- net MOSI: now also U3.28 (MOSI); no longer U3.27 (MISO)
- removed net GPIO13: U3.28 (MOSI), U4.J1_19 (GPIO13)
- net GPIO14 renamed SCLK
- new net: J5.A5 (CC1), R15.1
- new net: TP1.1, U3.55 (~{CS})
- new net: J5.B5 (CC2), R16.1
Other:
- note added: "+/-1%"

Commit message: ordering
Parts:
- added C4, C7: 10uF, Capacitor_SMD:C_0402_1005Metric, symbol Device:C_Small
- added C5, C6: 100nF, Capacitor_SMD:C_0402_1005Metric, symbol Device:C_Small
- D1, D2, D3, D4, D5, D6: footprint LED_SMD:LED_0201_0603Metric -> LED_SMD:LED_0603_1608Metric
Connections:
- net +3.3V: now also C4.1, C5.1, C6.1, C7.1
- net GND: now also C4.2, C5.2, C6.2, C7.2
